File: phq-u.kicad_pcb (KiCad board)
At the start: 4 copper layers, 130.4 x 75.4 mm, 102 parts, among them J1 18…56 V, J2 MCU bypass, J3 Voltage select, J4 3.3…24 V, J5 MCU disable, J6 TC2030, J7 USB-C, J8 I/O, Q1 NX138AK, U1 i7A4W033A033V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

Commit message: Add annotations to silkscreen
Parts:
- added G***: seal, LOGO, F.Cu at (181.5, 93.2)
- added G***: seal, LOGO, F.Cu at (120.0, 127.6)
- added G***: URL, LOGO, B.Cu at (179.8, 72.2)
- added REF**: Class_III, phq_Symbol:Class_III, B.Cu at (112.0, 127.7)
- added REF**: WEEE, phq_Symbol:WEEE, B.Cu at (102.0, 127.7)
Other:
- board text added: "+"
- board text added: "-"
- board text added: "Designed in 2022 by Mikael Voss This work may be used under the terms of the strictly‐reciprocative CERN Open Hardware Licence (CERN-OHL-S) version 2."
- board text added: "input 18-56 V⎓ 25 A"
- board text added: "output 3.3-24 V⎓ 30 A 500 W"
- board text added: "⏚"

Commit message: Invert project URL QR code
Parts:
- moved G*** 0.30 mm to (180.1, 72.2)
